File: proto/shield/shield.sch (KiCad schematic (older format))
At the start: 112 parts, among them J1 ESC_XY, J10 gpio_d, J11 gpio_d, J12 gpio_d, J13 gpio_d, J14 gpio_a, J15 gpio_a, J16 gpio_a, J17 gpio_a, J18 gpio_a, J19 gpio_a, J2 ESC_4Z, J20 gpio_a, J21 gpio_a, J22 5V_IN_A, J23 5V_IN_D, J3 PWM1, J4 PWM2, J5 PWM3, J6 gpio_d, J7 gpio_d, J8 gpio_d, J9 gpio_d, U1 NUCLEO144-F746ZG, U10 LTV-817S, U11 LTV-817S, U12 LTV-817S, U13 LTV-817S, U14 LTV-817S, U15 LTV-817S, U16 LTV-817S, U17 LTV-817S, U2 6N137, U3 6N137, U4 6N137, U5 6N137, U6 6N137, U7 6N137, U8 6N137, U9 6N137

Commit message: pcb + can + rs232
Parts:
- removed D?: >6, symbol Device:D_TVS
- removed U1: NUCLEO144-F746ZG, Module:ST_Morpho_Connector_144_STLink, symbol MCU_Module:NUCLEO144-F746ZG
- added C12, C17: 10u, Capacitor_SMD:C_0805_2012Metric, symbol Device:C
- added C13: 47n, Capacitor_SMD:C_0805_2012Metric, symbol Device:C
- added C14, C15, C16: 330n, Capacitor_SMD:C_0805_2012Metric, symbol Device:C
- added J24: CAN_LINK, Connector_Molex:Molex_MicroClasp_55932-0230_1x02_P2.00mm_Vertical, symbol Connector_Generic:Conn_01x02
- added J25: Conn_01x04, Connector_JST:JST_PH_B4B-PH-K_1x04_P2.00mm_Vertical, symbol Connector_Generic:Conn_01x04
- added R55: 2k2, Resistor_SMD:R_0805_2012Metric, symbol Device:R
- added R56: 10k, Resistor_SMD:R_0805_2012Metric, symbol Device:R
- added R57: 120, Resistor_SMD:R_0805_2012Metric, symbol Device:R
- added U1: NUCLEO144-F767ZI, Module:ST_Morpho_Connector_144_STLink, symbol NUCLEO-F767ZI:NUCLEO144-F767ZI
- added U18: SN65HVD230, Package_SO:SOIC-8_3.9x4.9mm_P1.27mm, symbol Interface_CAN_LIN:SN65HVD230
- added U19: MAX3232, Package_SO:SOIC-16_4.55x10.3mm_P1.27mm, symbol Interface_UART:MAX3232
- C10: renamed from C?; footprint (none) -> Capacitor_Tantalum_SMD:CP_EIA-3528-21_Kemet-B
- C11, C9: renamed from C?; footprint (none) -> Capacitor_SMD:C_0805_2012Metric
- gave numbers to parts that had none: 4
Connections:
- net +5V: now also U1.6 (E5V)
- net +5VD: now also C17.1, J25.1 (Pin_1), U1.18 (+5V), U19.16 (VCC)
- net GNDD: now also C12.2, C15.1, C16.1, C17.2, J25.4 (Pin_4), R56.1, U1.111 (GND), U1.126 (GND), U1.135 (GND), U1.143 (GND), U1.144 (GND), U1.19 (GND), U1.20 (GND), U1.22 (GND), U1.49 (GND), U1.60 (GND), U1.71 (GND), U1.72 (GND), U1.8 (GND), U1.81 (GND), U1.92 (GND), U18.2 (GND), U19.15 (GND)
- net IO1: now also U1.35 (PC2)
- net IO2: now also U1.37 (PC3)
- net IO3: now also U1.4 (PD2)
- net IO4: now also U1.40 (PD3)
- net IO5: now also U1.39 (PD4)
- net IO6: now also U1.42 (PG2)
- net IO7: now also U1.44 (PG3)
- net IO8: now also U1.45 (PD7)
- net LED1: now also U1.136 (PE0)
- net LED2: now also U1.61 (PE1)
- net LED3: now also U1.46 (PE2)
- net LED4: now also U1.47 (PE3)
- net TIM3_CH1: now also U1.83 (PA5)
- net TIM3_CH2: now also U1.96 (PB1)
- net TIM3_CH3: now also U1.91 (PC7)
- net TIM3_CH4: now also U1.74 (PC8)
- net TIM4_CH1: now also U1.115 (PD12)
- net TIM4_CH2: now also U1.113 (PD13)
- net TIM4_CH3: now also U1.118 (PD14)
- net TIM4_CH4: now also U1.120 (PD15)
- new net: R55.1, R56.2, U18.8 (Rs)
- new net: C13.1, U19.1 (C1+)
- new net: C15.2, U19.2 (VS+)
- new net: C13.2, U19.3 (C1-)
- new net: C14.1, U19.4 (C2+)
- new net: C14.2, U19.5 (C2-)
- new net: C16.2, U19.6 (VS-)
- new net +3V3: C12.1, R55.2, U1.16 (+3V3), U18.3 (VCC)
- new net CAN1_RX: U1.57 (PD0), U18.4 (R)
- new net CAN1_TX: U1.55 (PD1), U18.1 (D)
- new net CAN_H: J24.1 (Pin_1), R57.1, U18.7 (CANH)
- new net CAN_L: J24.2 (Pin_2), R57.2, U18.6 (CANL)
- new net RS232_RX: J25.3 (Pin_3), U19.13 (R1IN)
- new net RS232_TX: J25.2 (Pin_2), U19.14 (T1OUT)
- new net UART_RS_RX: U1.43 (PD6), U19.12 (R1OUT)
- new net UART_RS_TX: U1.41 (PD5), U19.11 (T1IN)
- no-connect marks 0 -> 5

Commit message: new layout
Connections:
- net IO1: now also U1.4 (PD2); no longer U1.35 (PC2)
- net IO2: now also U1.35 (PC2); no longer U1.37 (PC3)
- net IO3: now also U1.37 (PC3); no longer U1.4 (PD2)
- net IO4: now also U1.39 (PD4); no longer U1.40 (PD3)
- net IO5: now also U1.40 (PD3); no longer U1.39 (PD4)
- net TIM3_CH1: now also U1.74 (PC8); no longer U1.83 (PA5)
- net TIM3_CH2: now also U1.83 (PA5); no longer U1.96 (PB1)
- net TIM3_CH4: now also U1.96 (PB1); no longer U1.74 (PC8)
- net TIM4_CH1: now also U1.113 (PD13); no longer U1.115 (PD12)
- net TIM4_CH2: now also U1.115 (PD12); no longer U1.113 (PD13)
Changed lines of the file:
@@
 Comment4 ""
 $EndDescr
-Text Label 5625 4050 0    50   ~ 0
-TIM3_CH1
-Text Label 5625 5350 0    50   ~ 0
-TIM3_CH2
-Text Label 5625 9850 0    50   ~ 0
-TIM4_CH1
-Text Label 5625 9950 0    50   ~ 0
-TIM4_CH2
 Text Label 5625 10050 0    50   ~ 0
 TIM4_CH3
@@
 Wire Wire Line
 	5550 10150 5625 10150
-Text Label 5675 7150 0    50   ~ 0
+Text Label 5675 8850 0    50   ~ 0
 IO1
-Text Label 5675 7250 0    50   ~ 0
+Text Label 5675 7150 0    50   ~ 0
 IO2
-Text Label 5675 8850 0    50   ~ 0
+Text Label 5675 7250 0    50   ~ 0
 IO3
-Text Label 5675 8950 0    50   ~ 0
-IO4
 Text Label 5675 9050 0    50   ~ 0
+IO4
+Text Label 5675 8950 0    50   ~ 0
 IO5
 Text Label 2950 5450 2    50   ~ 0
@@
 	1    0    0    -1
 $EndComp
-Text Label 5650 7750 0    50   ~ 0
-TIM3_CH4
 Text Label 5650 7650 0    50   ~ 0
 TIM3_CH3
@@
 Wire Wire Line
 	15800 13225 15800 13275
+Text Label 5650 7750 0    50   ~ 0
+TIM3_CH1
+Text Label 5625 4050 0    50   ~ 0
+TIM3_CH2
+Text Label 5625 5350 0    50   ~ 0
+TIM3_CH4
+Text Label 5625 9950 0    50   ~ 0
+TIM4_CH1
+Text Label 5625 9850 0    50   ~ 0
+TIM4_CH2
 $EndSCHEMATC

Commit message: pa5->pa6
Connections:
- net TIM3_CH2: now also U1.85 (PA6); no longer U1.83 (PA5)
Changed lines of the file:
@@
 TIM4_CH4
 Wire Wire Line
-	5550 4050 5625 4050
+	5550 4150 5625 4150
 Wire Wire Line
 	5625 5350 5550 5350
@@
 Text Label 5650 7750 0    50   ~ 0
 TIM3_CH1
-Text Label 5625 4050 0    50   ~ 0
+Text Label 5625 4150 0    50   ~ 0
 TIM3_CH2
 Text Label 5625 5350 0    50   ~ 0

Commit message: finall pcb
Parts:
- D6, D7: value LED_B -> PWR
- J10: value gpio_d -> IO5
- J11: value gpio_d -> IO6
- J12: value gpio_d -> IO7
- J13: value gpio_d -> IO8
- J14: value gpio_a -> IO1_A
- J15: value gpio_a -> IO2_A
- J16: value gpio_a -> IO3_A
- J17: value gpio_a -> IO4_A
- J18: value gpio_a -> IO5_A
- J19: value gpio_a -> IO6_A
- J20: value gpio_a -> IO7_A
- J21: value gpio_a -> IO8_A
- J24: value CAN_LINK -> CAN
- J25: value Conn_01x04 -> RS232
- J6: value gpio_d -> IO1
- J7: value gpio_d -> IO2
- J8: value gpio_d -> IO3
- J9: value gpio_d -> IO4
- renumbered R57 to CAN_R1, R55 to CAN_R2, R56 to CAN_R3
Connections:
- net TIM3_CH1 renamed PWM_T1_IN
- net TIM3_CH1_A renamed PWM_T1
- net TIM3_CH2 renamed PWM_T2_IN
- net TIM3_CH2_A renamed PWM_T2
- net TIM3_CH3 renamed PWM_T3_IN
- net TIM3_CH3_A renamed PWM_T3
- net TIM3_CH4 renamed PWM_T4_IN
- net TIM3_CH4_A renamed PWM_T4
- net TIM4_CH1 renamed PWM_T5:T8_IN
- net TIM4_CH1_A renamed PWM_T5:T8
- net TIM4_CH2 renamed PWM_OPT1_IN
- net TIM4_CH2_A renamed PWM_OPT1
- net TIM4_CH3 renamed PWM_OPT2_IN
- net TIM4_CH3_A renamed PWM_OPT2
- net TIM4_CH4 renamed PWM_OPT3_IN
- net TIM4_CH4_A renamed PWM_OPT3

Commit message: Add resistors value
Parts:
- R1, R11, R12, R13, R17, R18, R19, R2, R20, R25, R26, R27, R28, R3, R4, R5: value R -> 400
- R10, R14, R15, R16, R6, R7, R8, R9: value R_Small -> 1k
- R21, R22, R23, R24, R29, R30, R31, R32: value R -> 10k
- R49, R50, R51, R52, R53, R54: value R -> 680
Changed lines of the file:
@@
 P 10425 3750
 F 0 "R6" H 10484 3797 50  0000 L CNN
-F 1 "R_Small" H 10484 3704 50  0000 L CNN
+F 1 "1k" H 10484 3704 50  0000 L CNN
 F 2 "Resistor_SMD:R_0805_2012Metric" H 10425 3750 50  0001 C CNN
 F 3 "~" H 10425 3750 50  0001 C CNN
@@
 P 9400 3800
 F 0 "R1" V 9190 3800 50  0000 C CNN
-F 1 "R" V 9283 3800 50  0000 C CNN
+F 1 "400" V 9283 3800 50  0000 C CNN
 F 2 "Resistor_SMD:R_0805_2012Metric" V 9330 3800 50  0001 C CNN
 F 3 "~" H 9400 3800 50  0001 C CNN
@@
 P 10425 4900
 F 0 "R7" H 10484 4947 50  0000 L CNN
-F 1 "R_Small" H 10484 4854 50  0000 L CNN
+F 1 "1k" H 10484 4854 50  0000 L CNN
 F 2 "Resistor_SMD:R_0805_2012Metric" H 10425 4900 50  0001 C CNN
 F 3 "~" H 10425 4900 50  0001 C CNN
@@
 P 9400 4950
 F 0 "R2" V 9190 4950 50  0000 C CNN
-F 1 "R" V 9283 4950 50  0000 C CNN
+F 1 "400" V 9283 4950 50  0000 C CNN
 F 2 "Resistor_SMD:R_0805_2012Metric" V 9330 4950 50  0001 C CNN
 F 3 "~" H 9400 4950 50  0001 C CNN
@@
 P 10425 6075
 F 0 "R8" H 10484 6122 50  0000 L CNN
-F 1 "R_Small" H 10484 6029 50  0000 L CNN
+F 1 "1k" H 10484 6029 50  0000 L CNN
 F 2 "Resistor_SMD:R_0805_2012Metric" H 10425 6075 50  0001 C CNN
 F 3 "~" H 10425 6075 50  0001 C CNN
@@
 P 9400 6125
 F 0 "R3" V 9190 6125 50  0000 C CNN
-F 1 "R" V 9283 6125 50  0000 C CNN
+F 1 "400" V 9283 6125 50  0000 C CNN
 F 2 "Resistor_SMD:R_0805_2012Metric" V 9330 6125 50  0001 C CNN
 F 3 "~" H 9400 6125 50  0001 C CNN
@@
 P 10425 7300
 F 0 "R9" H 10484 7347 50  0000 L CNN
-F 1 "R_Small" H 10484 7254 50  0000 L CNN
+F 1 "1k" H 10484 7254 50  0000 L CNN
 F 2 "Resistor_SMD:R_0805_2012Metric" H 10425 7300 50  0001 C CNN
 F 3 "~" H 10425 7300 50  0001 C CNN
@@
 P 9400 7350
 F 0 "R4" V 9190 7350 50  0000 C CNN
-F 1 "R" V 9283 7350 50  0000 C CNN
+F 1 "400" V 9283 7350 50  0000 C CNN
 F 2 "Resistor_SMD:R_0805_2012Metric" V 9330 7350 50  0001 C CNN
 F 3 "~" H 9400 7350 50  0001 C CNN
@@
 P 10425 8475
 F 0 "R10" H 10484 8522 50  0000 L CNN
-F 1 "R_Small" H 10484 8429 50  0000 L CNN
+F 1 "1k" H 10484 8429 50  0000 L CNN
 F 2 "Resistor_SMD:R_0805_2012Metric" H 10425 8475 50  0001 C CNN
 F 3 "~" H 10425 8475 50  0001 C CNN
@@
 P 9400 8525
 F 0 "R5" V 9190 8525 50  0000 C CNN
-F 1 "R" V 9283 8525 50  0000 C CNN
+F 1 "400" V 9283 8525 50  0000 C CNN
 F 2 "Resistor_SMD:R_0805_2012Metric" V 9330 8525 50  0001 C CNN
 F 3 "~" H 9400 8525 50  0001 C CNN
@@
 P 12975 3700
 F 0 "R14" H 13034 3747 50  0000 L CNN
-F 1 "R_Small" H 13034 3654 50  0000 L CNN
+F 1 "1k" H 13034 3654 50  0000 L CNN
 F 2 "Resistor_SMD:R_0805_2012Metric" H 12975 3700 50  0001 C CNN
 F 3 "~" H 12975 3700 50  0001 C CNN
@@
 P 11950 3750
 F 0 "R11" V 11740 3750 50  0000 C CNN
-F 1 "R" V 11833 3750 50  0000 C CNN
+F 1 "400" V 11833 3750 50  0000 C CNN
 F 2 "Resistor_SMD:R_0805_2012Metric" V 11880 3750 50  0001 C CNN
 F 3 "~" H 11950 3750 50  0001 C CNN
@@
 P 12975 4875
 F 0 "R15" H 13034 4922 50  0000 L CNN
-F 1 "R_Small" H 13034 4829 50  0000 L CNN
+F 1 "1k" H 13034 4829 50  0000 L CNN
 F 2 "Resistor_SMD:R_0805_2012Metric" H 12975 4875 50  0001 C CNN
 F 3 "~" H 12975 4875 50  0001 C CNN
@@
 P 11950 4925
 F 0 "R12" V 11740 4925 50  0000 C CNN
-F 1 "R" V 11833 4925 50  0000 C CNN
+F 1 "400" V 11833 4925 50  0000 C CNN
 F 2 "Resistor_SMD:R_0805_2012Metric" V 11880 4925 50  0001 C CNN
 F 3 "~" H 11950 4925 50  0001 C CNN
@@
 P 12975 6100
 F 0 "R16" H 13034 6147 50  0000 L CNN
-F 1 "R_Small" H 13034 6054 50  0000 L CNN
+F 1 "1k" H 13034 6054 50  0000 L CNN
 F 2 "Resistor_SMD:R_0805_2012Metric" H 12975 6100 50  0001 C CNN
 F 3 "~" H 12975 6100 50  0001 C CNN
@@
 P 11950 6150
 F 0 "R13" V 11740 6150 50  0000 C CNN
-F 1 "R" V 11833 6150 50  0000 C CNN
+F 1 "400" V 11833 6150 50  0000 C CNN
 F 2 "Resistor_SMD:R_0805_2012Metric" V 11880 6150 50  0001 C CNN
 F 3 "~" H 11950 6150 50  0001 C CNN
@@
 P 15650 1650
 F 0 "R17" V 15440 1650 50  0000 C CNN
-F 1 "R" V 15533 1650 50  0000 C CNN
+F 1 "400" V 15533 1650 50  0000 C CNN
 F 2 "Resistor_SMD:R_0805_2012Metric" V 15580 1650 50  0001 C CNN
 F 3 "~" H 15650 1650 50  0001 C CNN
@@
 P 16500 2050
 F 0 "R21" H 16430 2003 50  0000 R CNN
-F 1 "R" H 16430 2096 50  0000 R CNN
+F 1 "10k" H 16430 2096 50  0000 R CNN
 F 2 "Resistor_SMD:R_0805_2012Metric" V 16430 2050 50  0001 C CNN
 F 3 "~" H 16500 2050 50  0001 C CNN
@@
 P 15650 2750
 F 0 "R18" V 15440 2750 50  0000 C CNN
-F 1 "R" V 15533 2750 50  0000 C CNN
+F 1 "400" V 15533 2750 50  0000 C CNN
 F 2 "Resistor_SMD:R_0805_2012Metric" V 15580 2750 50  0001 C CNN
 F 3 "~" H 15650 2750 50  0001 C CNN
@@
 P 16500 3150
 F 0 "R22" H 16430 3103 50  0000 R CNN
-F 1 "R" H 16430 3196 50  0000 R CNN
+F 1 "10k" H 16430 3196 50  0000 R CNN
 F 2 "Resistor_SMD:R_0805_2012Metric" V 16430 3150 50  0001 C CNN
 F 3 "~" H 16500 3150 50  0001 C CNN
@@
 P 15650 3850
 F 0 "R19" V 15440 3850 50  0000 C CNN
-F 1 "R" V 15533 3850 50  0000 C CNN
+F 1 "400" V 15533 3850 50  0000 C CNN
 F 2 "Resistor_SMD:R_0805_2012Metric" V 15580 3850 50  0001 C CNN
 F 3 "~" H 15650 3850 50  0001 C CNN
@@
 P 16500 4250
 F 0 "R23" H 16430 4203 50  0000 R CNN
-F 1 "R" H 16430 4296 50  0000 R CNN
+F 1 "10k" H 16430 4296 50  0000 R CNN
 F 2 "Resistor_SMD:R_0805_2012Metric" V 16430 4250 50  0001 C CNN
 F 3 "~" H 16500 4250 50  0001 C CNN
@@
 P 15700 4950
 F 0 "R20" V 15490 4950 50  0000 C CNN
-F 1 "R" V 15583 4950 50  0000 C CNN
+F 1 "400" V 15583 4950 50  0000 C CNN
 F 2 "Resistor_SMD:R_0805_2012Metric" V 15630 4950 50  0001 C CNN
 F 3 "~" H 15700 4950 50  0001 C CNN
@@
 P 16550 5350
 F 0 "R24" H 16480 5303 50  0000 R CNN
-F 1 "R" H 16480 5396 50  0000 R CNN
+F 1 "10k" H 16480 5396 50  0000 R CNN
 F 2 "Resistor_SMD:R_0805_2012Metric" V 16480 5350 50  0001 C CNN
 F 3 "~" H 16550 5350 50  0001 C CNN
@@
 P 17350 1650
 F 0 "R25" V 17140 1650 50  0000 C CNN
-F 1 "R" V 17233 1650 50  0000 C CNN
+F 1 "400" V 17233 1650 50  0000 C CNN
 F 2 "Resistor_SMD:R_0805_2012Metric" V 17280 1650 50  0001 C CNN
 F 3 "~" H 17350 1650 50  0001 C CNN
@@
 P 18200 2050
 F 0 "R29" H 18130 2003 50  0000 R CNN
-F 1 "R" H 18130 2096 50  0000 R CNN
+F 1 "10k" H 18130 2096 50  0000 R CNN
 F 2 "Resistor_SMD:R_0805_2012Metric" V 18130 2050 50  0001 C CNN
 F 3 "~" H 18200 2050 50  0001 C CNN
@@
 P 17350 2750
 F 0 "R26" V 17140 2750 50  0000 C CNN
-F 1 "R" V 17233 2750 50  0000 C CNN
+F 1 "400" V 17233 2750 50  0000 C CNN
 F 2 "Resistor_SMD:R_0805_2012Metric" V 17280 2750 50  0001 C CNN
 F 3 "~" H 17350 2750 50  0001 C CNN
@@
 P 18200 3150
 F 0 "R30" H 18130 3103 50  0000 R CNN
-F 1 "R" H 18130 3196 50  0000 R CNN
+F 1 "10k" H 18130 3196 50  0000 R CNN
 F 2 "Resistor_SMD:R_0805_2012Metric" V 18130 3150 50  0001 C CNN
 F 3 "~" H 18200 3150 50  0001 C CNN
@@
 P 17350 3850
 F 0 "R27" V 17140 3850 50  0000 C CNN
-F 1 "R" V 17233 3850 50  0000 C CNN
+F 1 "400" V 17233 3850 50  0000 C CNN
 F 2 "Resistor_SMD:R_0805_2012Metric" V 17280 3850 50  0001 C CNN
 F 3 "~" H 17350 3850 50  0001 C CNN
@@
 P 18200 4250
 F 0 "R31" H 18130 4203 50  0000 R CNN
-F 1 "R" H 18130 4296 50  0000 R CNN
+F 1 "10k" H 18130 4296 50  0000 R CNN
 F 2 "Resistor_SMD:R_0805_2012Metric" V 18130 4250 50  0001 C CNN
 F 3 "~" H 18200 4250 50  0001 C CNN
@@
 P 17400 4950
 F 0 "R28" V 17190 4950 50  0000 C CNN
-F 1 "R" V 17283 4950 50  0000 C CNN
+F 1 "400" V 17283 4950 50  0000 C CNN
 F 2 "Resistor_SMD:R_0805_2012Metric" V 17330 4950 50  0001 C CNN
 F 3 "~" H 17400 4950 50  0001 C CNN
@@
 P 18250 5350
 F 0 "R32" H 18180 5303 50  0000 R CNN
-F 1 "R" H 18180 5396 50  0000 R CNN
+F 1 "10k" H 18180 5396 50  0000 R CNN
 F 2 "Resistor_SMD:R_0805_2012Metric" V 18180 5350 50  0001 C CNN
 F 3 "~" H 18250 5350 50  0001 C CNN
@@
 P 13700 7750
 F 0 "R49" V 13490 7750 50  0000 C CNN
-F 1 "R" V 13583 7750 50  0000 C CNN
+F 1 "680" V 13583 7750 50  0000 C CNN
 F 2 "Resistor_SMD:R_0805_2012Metric" V 13630 7750 50  0001 C CNN
 F 3 "~" H 13700 7750 50  0001 C CNN
@@
 P 14150 7750
 F 0 "R50" V 13940 7750 50  0000 C CNN
-F 1 "R" V 14033 7750 50  0000 C CNN
+F 1 "680" V 14033 7750 50  0000 C CNN
 F 2 "Resistor_SMD:R_0805_2012Metric" V 14080 7750 50  0001 C CNN
 F 3 "~" H 14150 7750 50  0001 C CNN
@@
 P 14600 7750
 F 0 "R51" V 14390 7750 50  0000 C CNN
-F 1 "R" V 14483 7750 50  0000 C CNN
+F 1 "680" V 14483 7750 50  0000 C CNN
 F 2 "Resistor_SMD:R_0805_2012Metric" V 14530 7750 50  0001 C CNN
 F 3 "~" H 14600 7750 50  0001 C CNN
@@
 P 15050 7750
 F 0 "R52" V 14840 7750 50  0000 C CNN
-F 1 "R" V 14933 7750 50  0000 C CNN
+F 1 "680" V 14933 7750 50  0000 C CNN
 F 2 "Resistor_SMD:R_0805_2012Metric" V 14980 7750 50  0001 C CNN
 F 3 "~" H 15050 7750 50  0001 C CNN
@@
 P 14350 9125
 F 0 "R53" V 14140 9125 50  0000 C CNN
-F 1 "R" V 14233 9125 50  0000 C CNN
+F 1 "680" V 14233 9125 50  0000 C CNN
 F 2 "Resistor_SMD:R_0805_2012Metric" V 14280 9125 50  0001 C CNN
 F 3 "~" H 14350 9125 50  0001 C CNN
@@
 P 15125 10300
 F 0 "R54" V 14915 10300 50  0000 C CNN
-F 1 "R" V 15008 10300 50  0000 C CNN
+F 1 "680" V 15008 10300 50  0000 C CNN
 F 2 "Resistor_SMD:R_0805_2012Metric" V 15055 10300 50  0001 C CNN
 F 3 "~" H 15125 10300 50  0001 C CNN
